File: ESPBrewRIMS_PCB/ESPBrewRIMS_PCB.kicad_sch (KiCad schematic)
At the start: 41 parts, among them J1 Conn_01x02, J10 Conn_01x02, J11 Conn_01x02, J12 Conn_01x02, J13 Conn_01x02, J14 Conn_01x02, J2 Conn_01x02, J3 Conn_01x02, J4 Digital LED, J5 Conn_01x05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

Commit message: Sent version to JLCPCB for print
Parts:
- removed C2: C_Small, symbol Device:C_Small
- removed F1: Fuse, symbol Device:Fuse
- removed U2: ~, symbol Library:AC2DC5V
- added H1, H2, H3, H4: MountingHole, MountingHole:MountingHole_3mm, symbol Mechanical:MountingHole
- added J10, J11, J12, J13, J8, J9: Conn_01x01_Pin, Connector_PinSocket_2.54mm:PinSocket_1x01_P2.54mm_Vertical, symbol Connector:Conn_01x01_Pin
- added R10, R18: 0, Resistor_SMD:R_0805_2012Metric_Pad1.20x1.40mm_HandSolder, symbol Device:R_Small_US
- C1: footprint (none) -> Capacitor_THT:CP_Radial_D8.0mm_P3.50mm
- C2: renamed from C3; footprint (none) -> Capacitor_SMD:C_0805_2012Metric_Pad1.18x1.45mm_HandSolder
- C3: renamed from C4; footprint (none) -> Capacitor_SMD:C_0805_2012Metric_Pad1.18x1.45mm_HandSolder
- C4: renamed from C8; footprint (none) -> Capacitor_SMD:C_0805_2012Metric_Pad1.18x1.45mm_HandSolder
- C5: footprint (none) -> Capacitor_SMD:C_0805_2012Metric_Pad1.18x1.45mm_HandSolder
- C6: renamed from C7; footprint (none) -> Capacitor_SMD:C_0805_2012Metric_Pad1.18x1.45mm_HandSolder
- J1: footprint (none) -> Connector_Molex:Molex_SL_171971-0002_1x02_P2.54mm_Vertical
- J14: renamed from J13; footprint (none) -> Connector_Molex:Molex_SL_171971-0002_1x02_P2.54mm_Vertical
- J15: renamed from J8; footprint (none) -> Connector_Molex:Molex_SL_171971-0005_1x05_P2.54mm_Vertical
- J16: renamed from J6; footprint (none) -> Connector_Molex:Molex_SL_171971-0005_1x05_P2.54mm_Vertical
- J17: renamed from J7; footprint (none) -> Connector_Molex:Molex_SL_171971-0002_1x02_P2.54mm_Vertical
- J18: renamed from J5; footprint (none) -> Connector_Molex:Molex_SL_171971-0005_1x05_P2.54mm_Vertical
- J19: renamed from J14; footprint (none) -> Connector_Molex:Molex_SL_171971-0002_1x02_P2.54mm_Vertical
- J2: renamed from J12; footprint (none) -> Connector_Molex:Molex_SL_171971-0002_1x02_P2.54mm_Vertical
- J20: renamed from J9; footprint (none) -> Connector_PinHeader_2.54mm:PinHeader_1x05_P2.54mm_Vertical
- J3: renamed from J2; footprint (none) -> Connector_Molex:Molex_SL_171971-0002_1x02_P2.54mm_Vertical
- J4: renamed from J3; footprint (none) -> Connector_Molex:Molex_SL_171971-0002_1x02_P2.54mm_Vertical
- J5: renamed from J10; footprint (none) -> Connector_Molex:Molex_SL_171971-0002_1x02_P2.54mm_Vertical
- J6: renamed from J11; footprint (none) -> Connector_Molex:Molex_SL_171971-0002_1x02_P2.54mm_Vertical
- J7: renamed from J4; footprint (none) -> Connector_Molex:Molex_SL_171971-0005_1x05_P2.54mm_Vertical
- R1: renamed from R14; footprint (none) -> Resistor_SMD:R_0805_2012Metric_Pad1.20x1.40mm_HandSolder
- R11: renamed from R12; footprint (none) -> Resistor_SMD:R_0805_2012Metric_Pad1.20x1.40mm_HandSolder
- R12: renamed from R11; footprint (none) -> Resistor_SMD:R_0805_2012Metric_Pad1.20x1.40mm_HandSolder
- R13: renamed from R7; footprint (none) -> Resistor_SMD:R_0805_2012Metric_Pad1.20x1.40mm_HandSolder
- R14: renamed from R10; footprint (none) -> Resistor_SMD:R_0805_2012Metric_Pad1.20x1.40mm_HandSolder
- R15: renamed from R9; footprint (none) -> Resistor_SMD:R_0805_2012Metric_Pad1.20x1.40mm_HandSolder
- R16: footprint (none) -> Resistor_SMD:R_0805_2012Metric_Pad1.20x1.40mm_HandSolder
- R17: renamed from R8; footprint (none) -> Resistor_SMD:R_0805_2012Metric_Pad1.20x1.40mm_HandSolder
- R2: renamed from R1; footprint (none) -> Resistor_SMD:R_0805_2012Metric_Pad1.20x1.40mm_HandSolder
- R3: renamed from R2; footprint (none) -> Resistor_SMD:R_0805_2012Metric_Pad1.20x1.40mm_HandSolder
- R4: renamed from R5; footprint (none) -> Resistor_SMD:R_0805_2012Metric_Pad1.20x1.40mm_HandSolder
- R5: renamed from R6; footprint (none) -> Resistor_SMD:R_0805_2012Metric_Pad1.20x1.40mm_HandSolder
- R6: renamed from R3; footprint (none) -> Resistor_SMD:R_0805_2012Metric_Pad1.20x1.40mm_HandSolder
- R7: renamed from R4; footprint (none) -> Resistor_SMD:R_0805_2012Metric_Pad1.20x1.40mm_HandSolder
- R8: renamed from R15; footprint (none) -> Resistor_SMD:R_0805_2012Metric_Pad1.20x1.40mm_HandSolder
- R9: renamed from R13; footprint (none) -> Resistor_SMD:R_0805_2012Metric_Pad1.20x1.40mm_HandSolder
- U1: footprint (none) -> ESPBrew:DIP-36_907_ELL
Connections:
- net 5V: now also J1.1 (Pin_1)
- net ENC_A: now also U1.19 (J3_GPIO46); no longer U1.36 (J3_GPIO46)
- net ENC_B: now also U1.20 (J3_GPIO45); no longer U1.35 (J3_GPIO45)
- net ENC_SW: now also U1.21 (J3_GPIO42); no longer U1.34 (J3_GPIO42)
- net EX_CLK: now also U1.32 (J3_GPIO48); no longer U1.23 (J3_GPIO48)
- net EX_DIO: now also U1.33 (J3_GPIO26); no longer U1.22 (J3_GPIO26)
- net EX_STB: now also U1.31 (J3_GPIO47); no longer U1.24 (J3_GPIO47)
- net GND: now also J1.2 (Pin_2), U1.36 (J3_GND); no longer U1.19 (J3_GND)
- net SW_EX1: now also U1.30 (J3_GPIO33), R10.1; no longer J14.2 (Pin_2), U1.25 (J3_GPIO33)
- net SW_EX2: now also U1.29 (J3_GPIO34), R18.1; no longer J19.2 (Pin_2), U1.26 (J3_GPIO34)
- net SW_MODE: now also U1.22 (J3_GPIO41); no longer U1.33 (J3_GPIO41)
- net TC_CS1: now also U1.25 (J3_GPIO38); no longer U1.30 (J3_GPIO38)
- net TC_CS2: now also U1.26 (J3_GPIO37); no longer U1.29 (J3_GPIO37)
- net TC_SCK: now also U1.24 (J3_GPIO39); no longer U1.31 (J3_GPIO39)
- net TC_SO: now also U1.23 (J3_GPIO40); no longer U1.32 (J3_GPIO40)
- net Vcc: now also U1.35 (J3_3V3a); no longer U1.20 (J3_3V3a)
- net at U1.10 (J2_GPIO20): now also J10.1 (Pin_1)
- net at U1.11 (J2_GPIO19): now also J11.1 (Pin_1)
- net at U1.27 (J3_GPIO36): now also J13.1 (Pin_1)
- net at U1.28 (J3_GPIO35): now also J12.1 (Pin_1)
- net at U1.8 (J2_GPIO0): now also J8.1 (Pin_1)
- net at U1.9 (J2_GPIO21): now also J9.1 (Pin_1)
- new net: J19.2 (Pin_2), R18.2
- new net: J14.2 (Pin_2), R10.2
Other:
- moved on the sheet: C1, D1, J14, J19, J2, J3, J4, J5, J6, J7, R1, R16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

Commit message: updated encoder cap values
Parts:
- C4, C5, C6: value 1uF -> 0.01uF
Changed lines of the file:
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@@
 			)
 		)
-		(property "Value" "1uF"
+		(property "Value" "0.01uF"
 			(at 248.92 152.4062 0)
 			(effects
@@
 			)
 		)
-		(property "Value" "1uF"
+		(property "Value" "0.01uF"
 			(at 251.46 134.6262 0)
 			(effects
@@
 			)
 		)
-		(property "Value" "1uF"
+		(property "Value" "0.01uF"
 			(at 248.92 144.7862 0)
 			(effects

Commit message: added AC sch
Other:
- added sheet AC Circuit (untitled.kicad_sch)
Changed lines of the file:
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@@
+		)
+	)
+	(sheet
+		(at 146.05 24.13)
+		(size 39.37 20.32)
+		(exclude_from_sim yes)
+		(in_bom no)
+		(on_board no)
+		(dnp yes)
+		(fields_autoplaced yes)
+		(stroke
+			(width 0.1524)
+			(type solid)
+		)
+		(fill
+			(color 0 0 0 0.0000)
+		)
+		(property "Sheetname" "AC Circuit"
+			(at 146.05 23.4184 0)
+			(effects
+				(font
+					(size 1.27 1.27)
+				)
+				(justify left bottom)
+			)
+		)
+		(property "Sheetfile" "untitled.kicad_sch"
+			(at 146.05 45.0346 0)
+			(effects
+				(font
+					(size 1.27 1.27)
+				)
+				(justify left top)
+			)
+		)
+		(instances
+			(project "ESPBrewRIMS_PCB"
+				(path "/d2ead811-201e-452d-a099-1da243f26c54"
+					(page "2")
+				)
+			)
 		)
 	)
